Commit message: fixed problem with braccio calibration

File: braccio_description/urdf/xacros/camera_and_mount_and_braccio.urdf.xacro (robot description, xacro)
@@ -8,5 +8,5 @@
     </xacro:camera_mount>
     <xacro:sensor_d435 parent="mount">
-        <origin xyz="0.0 0.0 0.6" rpy="0.0 1.0 1.10" />
+        <origin xyz="0.02 0.015 0.604" rpy="-0.02 1.00 1.58" />
     </xacro:sensor_d435>
     <xacro:kuka parent="mount">

File: braccio_description/urdf/xacros/camera_and_mount_and_braccio_planning.urdf.xacro (robot description, xacro)
@@ -8,5 +8,5 @@
     </xacro:camera_mount>
     <xacro:sensor_d435 parent="mount">
-        <origin xyz="0.0 0.0 0.625" rpy="0.0 1.10 1.10" />
+        <origin xyz="0.02 0.015 0.604" rpy="-0.02 1.00 1.58" />
     </xacro:sensor_d435>
     <xacro:kr5 parent="mount">

File: braccio_description/urdf/xacros/camera_mount_model.urdf.xacro (robot description, xacro)
@@ -10,5 +10,6 @@
             <visual>
                 <geometry>
-                    <mesh filename="package://braccio_description/stl/camera_mount.stl" scale="0.001 0.001 0.001"/>
+                    <!-- <mesh filename="package://braccio_description/stl/camera_mount.stl" scale="0.001 0.001 0.001"/> -->
+                    <mesh filename="package://braccio_description/stl/assieme.stl" scale="0.001 0.001 0.001"/>
                 </geometry>
                 <material name="white"/>
@@ -17,13 +18,14 @@
             <collision>
                 <geometry>
-                    <mesh filename="package://braccio_description/stl/camera_mount.stl" scale="0.001 0.001 0.001"/>
+                    <!-- <mesh filename="package://braccio_description/stl/camera_mount.stl" scale="0.001 0.001 0.001"/> -->
+                    <mesh filename="package://braccio_description/stl/assieme.stl" scale="0.001 0.001 0.001"/>
                 </geometry>
                 <origin rpy="1.57 0 0.78" xyz="0 0.0 0" />
             </collision>
         </link>
-        <joint name="mount_joint" type="continuous" >
+        <joint name="mount_joint" type="fixed" >
             <parent link="${parent}" />
             <child link="mount" />
-            <axis xyz="0 0 -1" />
+            <!-- <axis xyz="0 0 -1" /> -->
         </joint>
     </xacro:macro>

Commit message: added bounding box in PCL

File: braccio_description/urdf/xacros/camera_and_mount_and_braccio.urdf.xacro (robot description, xacro)
@@ -8,5 +8,6 @@
     </xacro:camera_mount>
     <xacro:sensor_d435 parent="mount">
-        <origin xyz="0.05 0.015 0.59" rpy="-0.12 1.15 0.780" />
+        <!-- <origin xyz="0.05 0.015 0.59" rpy="-0.12 1.15 0.780" /> -->
+        <origin xyz="0.05 0.015 0.59" rpy="-0.00 0.00 0.0" />
     </xacro:sensor_d435>
     <xacro:kuka parent="mount">

File: braccio_description/urdf/xacros/camera_and_mount_and_braccio_planning.urdf.xacro (robot description, xacro)
@@ -8,5 +8,6 @@
     </xacro:camera_mount>
     <xacro:sensor_d435 parent="mount">
-        <origin xyz="0.05 0.015 0.59" rpy="-0.12 1.15 0.780" />
+        <!-- <origin xyz="0.05 0.015 0.59" rpy="-0.12 1.15 0.780" /> -->
+        <origin xyz="0.05 0.015 0.59" rpy="-0.12 1.15 0.78" />
     </xacro:sensor_d435>
     <xacro:kr5 parent="mount">
