Commit message: changed start position

File: braccio_description/urdf/xacros/braccio_model.urdf.xacro (robot description, xacro)
@@ -179,5 +179,6 @@
                 <axis xyz="1 0 0" />
                 <limit effort="1.0" lower="0.2618" upper="2.8798" velocity="1.0" />
-                <origin rpy="-1.5708 0 0" xyz="0 -.002 0.072" />
+                <!-- <origin rpy="-1.587 0 0" xyz="0 -.002 0.072" /> -->
+                <origin rpy="2.0 0 0" xyz="0 -.002 0.072" />
                 <parent link="link_1" />
                 <child link="link_2" />

Commit message: added braccio_grasp_link tf

File: braccio_description/urdf/xacros/braccio_model.urdf.xacro (robot description, xacro)
@@ -314,4 +314,11 @@
             <axis xyz="0 0 -1" />
         </joint>
+        <!-- Fake joint and link for grasping -->
+	  	<joint name="braccio_grasp_joint" type="fixed">
+			<origin rpy="0 0 1.57" xyz="-0.06 0.03 0.16"/>
+			<parent link="left_gripper_link" />
+			<child link="gripper_grasp_link" />
+		</joint>
+		<link name="gripper_grasp_link"/>
      </xacro:macro>
 </robot>

File: braccio_description/urdf/xacros/braccio_model_planning.urdf.xacro (robot description, xacro)
@@ -329,4 +329,11 @@
         <child link="base_link"/>
     </joint>
+    <!-- Fake joint and link for grasping -->
+    <joint name="braccio_grasp_joint" type="fixed">
+        <origin rpy="0 1.835 0.0" xyz="0.09 0.0 -0.025"/>
+        <parent link="left_gripper_link" />
+        <child link="gripper_grasp_link" />
+    </joint>
+    <link name="gripper_grasp_link"/>
     </xacro:macro>
 </robot>

Commit message: modified joint angles and routin in go_to_xy method

File: braccio_description/urdf/xacros/braccio_model.urdf.xacro (robot description, xacro)
@@ -180,5 +180,5 @@
                 <limit effort="1.0" lower="0.2618" upper="2.8798" velocity="1.0" />
                 <!-- <origin rpy="-1.587 0 0" xyz="0 -.002 0.072" /> -->
-                <origin rpy="2.0 0 0" xyz="0 -.002 0.072" />
+                <origin rpy="2.0 0 0" xyz="0 -.002 0.1" />
                 <parent link="link_1" />
                 <child link="link_2" />

File: braccio_description/urdf/xacros/braccio_model_planning.urdf.xacro (robot description, xacro)
@@ -177,5 +177,5 @@
         <axis xyz="1 0 0" />
         <limit effort="1000.0" lower="0.2618" upper="2.8798" velocity="1.0" />
-        <origin rpy="-1.5708 0 0" xyz="0 -.002 0.072" />
+        <origin rpy="-1.5708 0 0" xyz="0 -.002 0.10" />
         <parent link="link_1" />
         <child link="link_2" />

File: braccio_description/urdf/xacros/camera_mount_model.urdf.xacro (robot description, xacro)
@@ -16,11 +16,11 @@
                 <origin rpy="1.57 0 0.78" xyz="0 0.0 0" />
             </visual>
-            <!-- <collision>
-                <geometry> -->
+            <collision>
+                <geometry>
                     <!-- <mesh filename="package://braccio_description/stl/camera_mount.stl" scale="0.001 0.001 0.001"/> -->
-                    <!-- <mesh filename="package://braccio_description/stl/assieme2.stl" scale="0.001 0.001 0.001"/>
+                   <mesh filename="package://braccio_description/stl/assieme2.stl" scale="0.001 0.001 0.001"/>
                 </geometry>
                 <origin rpy="1.57 0 0.78" xyz="0 0.0 0" />
-            </collision> -->
+            </collision>
         </link>
         <joint name="mount_joint" type="fixed" >

Commit message: merged targetter and braccio_model from pcl branch

File: braccio_description/urdf/xacros/braccio_model.urdf.xacro (robot description, xacro)
@@ -180,5 +180,5 @@
                 <limit effort="1.0" lower="0.2618" upper="2.8798" velocity="1.0" />
                 <!-- <origin rpy="-1.587 0 0" xyz="0 -.002 0.072" /> -->
-                <origin rpy="2.0 0 0" xyz="0 -.002 0.072" />
+                <origin rpy="2.0 0 0" xyz="0 -.002 0.1" />
                 <parent link="link_1" />
                 <child link="link_2" />
@@ -314,4 +314,11 @@
             <axis xyz="0 0 -1" />
         </joint>
+        <!-- Fake joint and link for grasping -->
+	  	<joint name="braccio_grasp_joint" type="fixed">
+			<origin rpy="0 0 1.57" xyz="-0.06 0.03 0.16"/>
+			<parent link="left_gripper_link" />
+			<child link="gripper_grasp_link" />
+		</joint>
+		<link name="gripper_grasp_link"/>
      </xacro:macro>
 </robot>

File: braccio_description/urdf/xacros/braccio_model_planning.urdf.xacro (robot description, xacro)
@@ -177,5 +177,5 @@
         <axis xyz="1 0 0" />
         <limit effort="1000.0" lower="0.2618" upper="2.8798" velocity="1.0" />
-        <origin rpy="-1.5708 0 0" xyz="0 -.002 0.072" />
+        <origin rpy="-1.5708 0 0" xyz="0 -.002 0.10" />
         <parent link="link_1" />
         <child link="link_2" />
@@ -329,4 +329,11 @@
         <child link="base_link"/>
     </joint>
+    <!-- Fake joint and link for grasping -->
+    <joint name="braccio_grasp_joint" type="fixed">
+        <origin rpy="0 1.835 0.0" xyz="0.09 0.0 -0.025"/>
+        <parent link="left_gripper_link" />
+        <child link="gripper_grasp_link" />
+    </joint>
+    <link name="gripper_grasp_link"/>
     </xacro:macro>
 </robot>

Commit message: changed grasp link names, reached minimum position_tolerance and set orientation_tolerance

File: braccio_description/urdf/xacros/braccio_model.urdf.xacro (robot description, xacro)
@@ -168,4 +168,24 @@
                 </collision>
             </link>
+            <link name="central_gripper_link">
+                <!-- <visual>
+                    <geometry>
+                        <mesh filename="package://braccio_description/stl/braccio_right_gripper.stl" scale="0.001 0.001 0.001" />
+                    </geometry>
+                    <material name="white" />
+                    <origin rpy="0 1.5708 0" xyz="0 -0.012 0.010" />
+                </visual> -->
+                <inertial>
+                    <origin rpy="0 0 0" xyz="0.043 0.001 0.002" />
+                    <mass value="0.01" />
+                    <inertia ixx="0.000348958333333" ixy="0" ixz="0" iyy="0.000348958333333" iyz="0" izz="3.125e-05" />
+                </inertial>
+                <!-- <collision>
+                    <origin rpy="0 1.5708 0" xyz="0 -0.012 0.010" />
+                    <geometry>
+                        <mesh filename="package://braccio_description/stl/braccio_right_gripper.stl" scale="0.001 0.001 0.001" />
+                    </geometry>
+                </collision> -->
+                </link>
             <joint name="base_joint" type="revolute">
                 <axis xyz="0 0 -1" />
@@ -315,10 +335,31 @@
         </joint>
         <!-- Fake joint and link for grasping -->
-	  	<joint name="braccio_grasp_joint" type="fixed">
-			<origin rpy="0 0 1.57" xyz="-0.06 0.03 0.16"/>
-			<parent link="left_gripper_link" />
-			<child link="gripper_grasp_link" />
-		</joint>
-		<link name="gripper_grasp_link"/>
+        <joint name="braccio_grasp_joint" type="continuous">
+            <origin rpy="0 0 0.0" xyz="0.0 0.0 0.04"/>
+            <parent link="link_5" />
+            <child link="arm_grasp_link" />
+        </joint>
+		<link name="arm_grasp_link">
+        <!-- <collision>
+        <origin xyz="0 0 0" rpy="0 0 0" />
+        <geometry>
+            <cylinder length="0.001" radius="0.001" />
+        </geometry>
+        </collision> -->
+        <inertial>
+            <origin xyz="0 0 0" rpy="0 0 0" />
+            <mass value="0.0001" />
+            <inertia
+            ixx="0.1" ixy="0.0" ixz="0.0"
+            iyy="0.10" iyz="0.0"
+            izz="0.1" />
+        </inertial>
+        </link>
+        <!-- Fake joint and link for gripper grasping -->
+        <joint name="gripper_grasp_joint" type="fixed">
+            <origin rpy="0 0 0.0" xyz="0.00 0.0 0.09"/>
+            <parent link="arm_grasp_link" />
+            <child link="central_gripper_link" />
+        </joint>
      </xacro:macro>
 </robot>

File: braccio_description/urdf/xacros/braccio_model_planning.urdf.xacro (robot description, xacro)
@@ -165,4 +165,24 @@
             </geometry>
         </collision>
+    </link>
+    <link name="central_gripper_link">
+        <!-- <visual>
+            <geometry>
+                <mesh filename="package://braccio_description/stl/braccio_right_gripper.stl" scale="0.001 0.001 0.001" />
+            </geometry>
+            <material name="white" />
+            <origin rpy="0 1.5708 0" xyz="0 -0.012 0.010" />
+        </visual> -->
+        <inertial>
+            <origin rpy="0 0 0" xyz="0.043 0.001 0.002" />
+            <mass value="0.01" />
+            <inertia ixx="0.000348958333333" ixy="0" ixz="0" iyy="0.000348958333333" iyz="0" izz="3.125e-05" />
+        </inertial>
+        <!-- <collision>
+            <origin rpy="0 1.5708 0" xyz="0 -0.012 0.010" />
+            <geometry>
+                <mesh filename="package://braccio_description/stl/braccio_right_gripper.stl" scale="0.001 0.001 0.001" />
+            </geometry>
+        </collision> -->
     </link>
     <joint name="base_joint" type="revolute">
@@ -341,9 +361,9 @@
     <!-- Fake joint and link for grasping -->
     <joint name="braccio_grasp_joint" type="continuous">
-        <origin rpy="0 0 0.0" xyz="0.0 0.0 0.03"/>
+        <origin rpy="0 0 0.0" xyz="0.0 0.0 0.04"/>
         <parent link="link_5" />
-        <child link="gripper_grasp_link" />
-    </joint>
-    <link name="gripper_grasp_link">
+        <child link="arm_grasp_link" />
+    </joint>
+    <link name="arm_grasp_link">
         <!-- <collision>
         <origin xyz="0 0 0" rpy="0 0 0" />
@@ -361,4 +381,10 @@
         </inertial>
         </link>
+    <!-- Fake joint and link for gripper grasping -->
+    <joint name="gripper_grasp_joint" type="fixed">
+        <origin rpy="0 0 0.0" xyz="0.00 0.0 0.09"/>
+        <parent link="arm_grasp_link" />
+        <child link="central_gripper_link" />
+    </joint>
     </xacro:macro>
 </robot>
