Commit message: working pose goal with braccio_grasp_joint physical properties

File: braccio_description/urdf/xacros/braccio_model_planning.urdf.xacro (robot description, xacro)
@@ -301,4 +301,14 @@
         </actuator>
     </transmission>
+    <transmission name="braccio_grasp_trans">
+        <type>transmission_interface/SimpleTransmission</type>
+        <joint name="braccio_grasp_joint">
+        <hardwareInterface>hardware_interface/EffortJointInterface</hardwareInterface>
+        </joint>
+        <actuator name="braccio_grasp_motor">
+        <hardwareInterface>hardware_interface/EffortJointInterface</hardwareInterface>
+        <mechanicalReduction>1</mechanicalReduction>
+        </actuator>
+    </transmission>
     <gazebo reference="link_1">
         <material>Gazebo/Green</material>
@@ -330,10 +340,25 @@
     </joint>
     <!-- Fake joint and link for grasping -->
-    <joint name="braccio_grasp_joint" type="fixed">
-        <origin rpy="0 1.835 0.0" xyz="0.09 0.0 -0.025"/>
-        <parent link="left_gripper_link" />
+    <joint name="braccio_grasp_joint" type="continuous">
+        <origin rpy="0 0 0.0" xyz="0.0 0.0 0.115"/>
+        <parent link="link_5" />
         <child link="gripper_grasp_link" />
     </joint>
-    <link name="gripper_grasp_link"/>
+    <link name="gripper_grasp_link">
+        <!-- <collision>
+        <origin xyz="0 0 0" rpy="0 0 0" />
+        <geometry>
+            <cylinder length="0.001" radius="0.001" />
+        </geometry>
+        </collision> -->
+        <inertial>
+            <origin xyz="0 0 0" rpy="0 0 0" />
+            <mass value="0.0001" />
+            <inertia
+            ixx="0.1" ixy="0.0" ixz="0.0"
+            iyy="0.10" iyz="0.0"
+            izz="0.1" />
+        </inertial>
+        </link>
     </xacro:macro>
 </robot>

Commit message: KDL position_tolerance to 0.12

File: braccio_description/urdf/xacros/braccio_model_planning.urdf.xacro (robot description, xacro)
@@ -341,5 +341,5 @@
     <!-- Fake joint and link for grasping -->
     <joint name="braccio_grasp_joint" type="continuous">
-        <origin rpy="0 0 0.0" xyz="0.0 0.0 0.115"/>
+        <origin rpy="0 0 0.0" xyz="0.0 0.0 0.03"/>
         <parent link="link_5" />
         <child link="gripper_grasp_link" />

Commit message: added targetter_pose_subscriber.py

File: braccio_description/urdf/xacros/braccio_model_planning.urdf.xacro (robot description, xacro)
@@ -361,5 +361,5 @@
     <!-- Fake joint and link for grasping -->
     <joint name="braccio_grasp_joint" type="continuous">
-        <origin rpy="0 0 0.0" xyz="0.0 0.0 0.04"/>
+        <origin rpy="0 0 0.0" xyz="0.0 0.0 0.115"/>
         <parent link="link_5" />
         <child link="arm_grasp_link" />
@@ -383,5 +383,5 @@
     <!-- Fake joint and link for gripper grasping -->
     <joint name="gripper_grasp_joint" type="fixed">
-        <origin rpy="0 0 0.0" xyz="0.00 0.0 0.09"/>
+        <origin rpy="0 0 0.0" xyz="0.00 0.0 0.015"/>
         <parent link="arm_grasp_link" />
         <child link="central_gripper_link" />

Commit message: moved tf_create in pose_goal_targetter

File: braccio_description/urdf/xacros/braccio_model_planning.urdf.xacro (robot description, xacro)
@@ -361,4 +361,7 @@
     <!-- Fake joint and link for grasping -->
     <joint name="braccio_grasp_joint" type="continuous">
+        <!-- <axis xyz="0 0 1" /> -->
+        <!-- <limit effort="10.0" lower="0.1750" upper="1.2741" velocity="1.0" />
+        <dynamics damping="0.1" friction="0.001" /> -->
         <origin rpy="0 0 0.0" xyz="0.0 0.0 0.115"/>
         <parent link="link_5" />

Commit message: somehow aligned with main

File: braccio_description/urdf/xacros/braccio_model_planning.urdf.xacro (robot description, xacro)
@@ -144,4 +144,15 @@
                 <mesh filename="package://braccio_description/stl/braccio_left_gripper.stl" scale="0.001 0.001 0.001" />
             </geometry>
+            <surface>
+                <friction>
+                    <ode>
+                    <mu>2000</mu>
+                    <mu2>1000</mu2>
+                    </ode>
+                    <torsional>
+                    <ode/>
+                    </torsional>
+                </friction>
+            </surface>
         </collision>
     </link>
@@ -164,4 +175,15 @@
                 <mesh filename="package://braccio_description/stl/braccio_right_gripper.stl" scale="0.001 0.001 0.001" />
             </geometry>
+            <surface>
+                <friction>
+                    <ode>
+                    <mu>2000</mu>
+                    <mu2>1000</mu2>
+                    </ode>
+                    <torsional>
+                    <ode/>
+                    </torsional>
+                </friction>
+            </surface>
         </collision>
     </link>
@@ -361,5 +383,8 @@
     <!-- Fake joint and link for grasping -->
     <joint name="braccio_grasp_joint" type="continuous">
-        <origin rpy="0 0 0.0" xyz="0.0 0.0 0.04"/>
+        <!-- <axis xyz="0 0 1" /> -->
+        <!-- <limit effort="10.0" lower="0.1750" upper="1.2741" velocity="1.0" />
+        <dynamics damping="0.1" friction="0.001" /> -->
+        <origin rpy="0 0 0.0" xyz="0.0 0.0 0.115"/>
         <parent link="link_5" />
         <child link="arm_grasp_link" />
@@ -383,5 +408,5 @@
     <!-- Fake joint and link for gripper grasping -->
     <joint name="gripper_grasp_joint" type="fixed">
-        <origin rpy="0 0 0.0" xyz="0.00 0.0 0.09"/>
+        <origin rpy="0 0 0.0" xyz="0.00 0.0 0.015"/>
         <parent link="arm_grasp_link" />
         <child link="central_gripper_link" />
