Commit message: added new mount and camera orientation

File: braccio_description/urdf/xacros/_d435.urdf.xacro (robot description, xacro)
@@ -44,13 +44,13 @@
     </joint>
     <link name="${name}_link">
-      <visual>
+      <!-- <visual>
       <origin xyz="${d435_cam_mount_from_center_offset} ${-d435_cam_depth_py} 0" rpy="${M_PI/2} 0 ${M_PI/2}"/>
-        <geometry>
+        <geometry> -->
           <!-- <box size="${d435_cam_width} ${d435_cam_height} ${d435_cam_depth}"/> -->
           <mesh filename="$(find realsense2_description)/meshes/d435.dae" />
           <!-- <mesh filename="package://realsense2_description/meshes/d435/d435.dae" /> -->
-        </geometry>
+        <!-- </geometry>
         <material name="${name}_aluminum"/>
-      </visual>
+      </visual> -->
       <collision>
         <origin xyz="0 ${-d435_cam_depth_py} 0" rpy="0 0 0"/>

File: braccio_description/urdf/xacros/camera_and_mount_and_braccio.urdf.xacro (robot description, xacro)
@@ -8,5 +8,5 @@
     </xacro:camera_mount>
     <xacro:sensor_d435 parent="mount">
-        <origin xyz="0.02 0.015 0.604" rpy="-0.02 1.00 1.58" />
+        <origin xyz="0.05 0.015 0.59" rpy="-0.12 1.15 0.780" />
     </xacro:sensor_d435>
     <xacro:kuka parent="mount">

File: braccio_description/urdf/xacros/camera_and_mount_and_braccio_planning.urdf.xacro (robot description, xacro)
@@ -8,5 +8,5 @@
     </xacro:camera_mount>
     <xacro:sensor_d435 parent="mount">
-        <origin xyz="0.02 0.015 0.604" rpy="-0.02 1.00 1.58" />
+        <origin xyz="0.05 0.015 0.59" rpy="-0.12 1.15 0.780" />
     </xacro:sensor_d435>
     <xacro:kr5 parent="mount">

File: braccio_description/urdf/xacros/camera_mount_model.urdf.xacro (robot description, xacro)
@@ -16,11 +16,11 @@
                 <origin rpy="1.57 0 0.78" xyz="0 0.0 0" />
             </visual>
-            <collision>
-                <geometry>
+            <!-- <collision>
+                <geometry> -->
                     <!-- <mesh filename="package://braccio_description/stl/camera_mount.stl" scale="0.001 0.001 0.001"/> -->
-                    <mesh filename="package://braccio_description/stl/assieme.stl" scale="0.001 0.001 0.001"/>
+                    <!-- <mesh filename="package://braccio_description/stl/assieme2.stl" scale="0.001 0.001 0.001"/>
                 </geometry>
                 <origin rpy="1.57 0 0.78" xyz="0 0.0 0" />
-            </collision>
+            </collision> -->
         </link>
         <joint name="mount_joint" type="fixed" >

Commit message: xacros modified

File: braccio_description/urdf/xacros/_d435.urdf.xacro (robot description, xacro)
@@ -48,5 +48,5 @@
         <geometry> -->
           <!-- <box size="${d435_cam_width} ${d435_cam_height} ${d435_cam_depth}"/> -->
-          <mesh filename="$(find realsense2_description)/meshes/d435.dae" />
+          <!-- <mesh filename="$(find realsense2_description)/meshes/d435.dae" /> -->
           <!-- <mesh filename="package://realsense2_description/meshes/d435/d435.dae" /> -->
         <!-- </geometry>

File: braccio_description/urdf/xacros/braccio_model.urdf.xacro (robot description, xacro)
@@ -329,5 +329,5 @@
                 <!-- <axis xyz="0 0 1"> -->
             <!-- </joint>  -->
-        <joint name="robot_joint" type="contiuous" >
+        <joint name="robot_joint" type="fixed" >
             <parent link="${parent}" />
             <child link="base_link" />
